File: pcb/FSKO-70-21-C.kicad_pcb (KiCad board)
At the start: 2 copper layers, 259 x 110.6 mm, 164 parts, among them J1 DX07S016JA3, J2 2x3_F, SW1 SW_Push, SW10 SW_Push, SW11 SW_Push, SW12 SW_Push, SW13 SW_Push, SW14 SW_Push, SW15 SW_Push, SW16 SW_Push, SW17 SW_Push, SW18 SW_Push, SW19 SW_Push, SW2 SW_Push, SW20 SW_Push, SW21 SW_Push, SW22 SW_Push, SW23 SW_Push, SW24 SW_Push, SW25 SW_Push, SW26 SW_Push, SW27 SW_Push, SW28 SW_Push, SW29 SW_Push, SW3 SW_Push, SW30 SW_Push, SW31 SW_Push, SW32 SW_Push, SW33 SW_Push, SW34 SW_Push, SW35 SW_Push, SW36 SW_Push, SW37 SW_Push, SW38 SW_Push, SW39 SW_Push, SW4 SW_Push, SW40 SW_Push, SW41 SW_Push, SW42 SW_Push, SW43 SW_Push, SW44 SW_Push, SW45 SW_Push, SW46 SW_Push, SW47 SW_Push, SW48 SW_Push, SW49 SW_Push, SW5 SW_Push, SW50 SW_Push, SW51 SW_Push, SW52 SW_Push, SW53 SW_Push, SW54 SW_Push, SW55 SW_Push, SW56 SW_Push, SW57 SW_Push, SW58 SW_Push, SW59 SW_Push, SW6 SW_Push, SW60 SW_Push, SW61 SW_Push, SW62 SW_Push, SW63 SW_Push, SW64 SW_Push, SW65 SW_Push, SW66 SW_Push, SW67 SW_Push, SW68 SW_Push, SW69 SW_Push, SW7 SW_Push, SW70 SW_Push, SW71 SW_Push, SW8 SW_Push, SW9 SW_Push, U1 ATmega32U4-AU, Y1 16MHz

Commit message: :sparkles: change key switch
Parts:
- SW1, SW10, SW11, SW12, SW13, SW14, SW15, SW16, SW17, SW18, SW19, SW2, SW20, SW21, SW22, SW23, SW24, SW25, SW26, SW27, SW28, SW29, SW3, SW30, SW31, SW32, SW33, SW34, SW35, SW36, SW37, SW38, SW39, SW4, SW40, SW41, SW42, SW43, SW44, SW45, SW46, SW47, SW48, SW49, SW5, SW50, SW51, SW52, SW53, SW54, SW55, SW56, SW57, SW58, SW59, SW6, SW60, SW61, SW62, SW63, SW64, SW65, SW66, SW67, SW68, SW69, SW7, SW70, SW8, SW9: footprint keyboard_toms:CherryMX_Choc_V2_1u -> keyboard_toms:Choc_V1_1u; moved to F.Cu
- moved D57 248.6 mm to (92.7, 220.6), turned to 0 degrees
- moved D1 247.9 mm to (92.7, 152.4), turned to 0 degrees
- moved SW1 247.9 mm to (92.7, 147.3)
- moved SW15 247.8 mm to (92.7, 164.3), turned to 0 degrees
- moved D15 247.8 mm to (92.7, 169.9), turned to 0 degrees
- moved D29 247.8 mm to (92.7, 187.4), turned to 0 degrees
- moved SW29 247.8 mm to (92.7, 181.3), turned to 0 degrees
- moved D43 247.7 mm to (92.7, 203.7), turned to 0 degrees
- moved SW43 247.7 mm to (92.7, 198.3), turned to 0 degrees
- moved SW57 247.7 mm to (92.7, 215.3), turned to 0 degrees
- moved D14 228.1 mm to (326.9, 152.4), turned to 0 degrees
- moved D28 228.0 mm to (326.9, 169.9), turned to 0 degrees
- moved D42 228.0 mm to (326.9, 187.4), turned to 0 degrees
- moved D56 227.9 mm to (326.9, 203.7), turned to 0 degrees
- moved D70 227.9 mm to (326.9, 220.6), turned to 0 degrees
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Connections:
- Y1 pad 2: (no net) -> Net-(C4-Pad1)
- Y1 pad 3: Net-(C4-Pad1) -> (no net)
Other:
- board size 259 x 110.6 mm -> 260 x 110.6 mm
